File: docmentation/eagle/LR_meter.sch (EAGLE design)
At the start: 0 parts

Commit message: version 1.0-1
Parts:
- added C1, C2: 1uF, capacitor-wima:C5/2.5
- added D1: 1N4148DO35-10, diode:1N4148DO35-10
- added IC1: LM393N, linear:LM393N
- added INDUCTORTEST, RESISTORTEST2: 0, con-wago-500:W237-102
- added R1: 1K, eagle-ltspice:R0207/10
- added R2: 2K, eagle-ltspice:R0207/10
- added R3: 20k, eagle-ltspice:R0207/10
- added R4: 200k, eagle-ltspice:R0207/10
- added R5: 1M, eagle-ltspice:R0207/10
- added R6: 150, eagle-ltspice:R0207/10
- added R7: 330, resistor:R-EU_0207/15
- added U$1: NANO, Arduino-clone:NANO
- added X1: 22-23-2051, con-molex:22-23-2051
Connections:
- new net 5V: IC1P.V+, R7.1, U$1.5.5V, X1-1.S
- new net GND: C1.2, C2.2, IC1A.-IN, IC1P.V-, INDUCTORTEST-2.KL, R1.2, U$1.GND
- new net N$11: RESISTORTEST2-2.KL, U$1.D7
- new net N$12: R6.1, U$1.D13
- new net N$13: C1.1, C2.1, D1.C, IC1A.+IN
- new net N$14: D1.A, R6.2
- new net N$15: IC1A.OUT, INDUCTORTEST-1.KL, R7.2
- new net N$2: U$1.A0, X1-2.S
- new net N$3: U$1.A1, X1-3.S
- new net N$30: R2.2, R3.1, R4.2, R5.2, RESISTORTEST2-1.KL, U$1.A2
- new net N$4: R1.1, U$1.D2, X1-4.S
- new net N$5: U$1.GND2, X1-5.S
- new net N$6: R2.1, U$1.D11
- new net N$7: R3.2, U$1.D10
- new net N$8: R4.1, U$1.D9
- new net N$9: R5.1, U$1.D8
Other:
- note added: "joystick"
